Commit message: PI -> M_PI

File: urdf/indoornav_husky.urdf.xacro (robot description, xacro)
@@ -7,5 +7,5 @@
       <parent link="base_link" />
       <child link="upgraded_imu_link" />
-      <origin xyz="0 0 0" rpy="0 0 ${PI}" />
+      <origin xyz="0 0 0" rpy="0 0 ${M_PI}" />
     </joint>
   </xacro:if>
@@ -14,5 +14,5 @@
       <parent link="base_link" />
       <child link="upgraded_imu_link" />
-      <origin xyz="0 0 0" rpy="0 0 ${PI/2}" />
+      <origin xyz="0 0 0" rpy="0 0 ${M_PI/2}" />
     </joint>
   </xacro:unless>
